File: eagle/Orange-Pi-Zero/Pixel/P2/zero_board.brd (EAGLE design)
At the start: 47.8 x 46 mm, 13 parts, among them CN1 1X4-3.5MM, IC1 74HCT125N, J1 1X2-3.5MM

Commit message: Removed pixel driver prototype V1
Parts:
- IC1: value 74HCT125N -> 74HCT125
Changed lines of the file:
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@@
 <element name="CN1" library="adafruit" package="1X04-3.5MM" value="1X4-3.5MM" x="5.08" y="24.384" rot="R270"/>
 <element name="J1" library="adafruit" package="1X2-3.5MM" value="1X2-3.5MM" x="5.08" y="36.068" rot="R270"/>
-<element name="IC1" library="74xx-eu" package="DIL14" value="74HCT125N" x="27.94" y="15.748" rot="R90"/>
+<element name="IC1" library="74xx-eu" package="DIL14" value="74HCT125" x="27.94" y="15.748" rot="R90"/>
 <element name="R2" library="rcl" package="0204/7" value="" x="19.05" y="18.288" rot="R90"/>
 <element name="C2" library="rcl" package="E5-6" value="" x="12.7" y="36.83" rot="R90"/>
@@
 <wire x1="40.386" y1="42.418" x2="40.386" y2="44.196" width="0.4064" layer="1"/>
 <wire x1="26.67" y1="26.924" x2="26.67" y2="34.29" width="0.6096" layer="1"/>
-<wire x1="27.94" y1="18.288" x2="27.432" y2="18.288" width="0" layer="19" extent="1-16"/>
-<wire x1="27.432" y1="18.288" x2="26.416" y2="18.288" width="0" layer="19" extent="1-16"/>
 <wire x1="27.94" y1="18.288" x2="24.13" y2="18.288" width="0.6096" layer="16"/>
-<wire x1="26.67" y1="18.542" x2="26.416" y2="18.288" width="0" layer="19" extent="1-16"/>
 <wire x1="24.13" y1="8.128" x2="27.432" y2="8.128" width="0.6096" layer="16"/>
 <wire x1="27.432" y1="8.128" x2="27.94" y2="8.636" width="0.6096" layer="16"/>

Commit message: Updates
Work in progress -> http://www.orangepi-dmx.org/pixel-boards
Parts:
- removed I2C: (no value), con-lstb:MA04-1
- added SV2: OPi Zero 2x13, con-lsta:FE13-2
- C1, C2: value (none) -> 1000u
- C3: value (none) -> 100n
- JP1: value (none) -> jumper
- LED1: value (none) -> 3mm
- R1, R2: value (none) -> 330
- SV1: value (none) -> OPi Zero 1x13
- SV3: value (none) -> I2C-OLED; device con-lsta:FE13-2 -> con-lstb:MA04-1
- moved R1 22.4 mm to (19.1, 18.3), turned to 90 degrees
- moved R2 22.4 mm to (27.9, 38.9), turned to 180 degrees
- moved SV3 22.2 mm to (5.08, 11.7), flipped to the top, turned to 270 degrees
- renumbered SV4 to SV1
Connections:
- removed net SPI_MISO: SV3.21
- net 3V3: now also SV2.1, SV3.2; no longer I2C.2, SV3.1
- net 5V: now also SV2.2, SV2.4; no longer SV3.2, SV3.4
- net GND: now also R2.1, SV2.14, SV2.20, SV2.25, SV2.6, SV2.9, SV3.1; no longer I2C.1, R1.1, SV3.14, SV3.20, SV3.25, SV3.6, SV3.9
- net I2C_SCL: now also SV2.5, SV3.3; no longer I2C.3, SV3.5
- net I2C_SDA: now also SV2.3, SV3.4; no longer I2C.4, SV3.3
- net MOSI: now also R1.1; no longer R2.1
- net N$1: now also R2.2; no longer R1.2
- net N$2: now also R1.2; no longer R2.2
- net SPI_CLK: now also SV2.23; no longer SV3.23
- net SPI_MOSI: now also SV2.19; no longer SV3.19
Changed lines of the file:
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@@
 <?xml version="1.0" encoding="utf-8"?>
 <!DOCTYPE eagle SYSTEM "eagle.dtd">
-<eagle version="6.4">
+<eagle version="6.6.0">
 <drawing>
 <settings>
@@
 </autorouter>
 <elements>
-<element name="SV4" library="con-lsta" package="FE13" value="" x="25.146" y="44.196" rot="MR0">
+<element name="SV1" library="con-lsta" package="FE13" value="OPi Zero 1x13" x="25.146" y="44.196" rot="MR0">
 <attribute name="OC_NEWARK" value="unknown" x="25.146" y="44.196" size="1.778" layer="28" rot="MR0" display="off"/>
 <attribute name="MPN" value="" x="25.146" y="44.196" size="1.778" layer="28" rot="MR0" display="off"/>
@@
 <attribute name="OC_FARNELL" value="unknown" x="25.146" y="44.196" size="1.778" layer="28" rot="MR0" display="off"/>
 </element>
-<element name="SV3" library="con-lsta" package="FE13-2" value="" x="25.146" y="2.286" rot="MR180">
+<element name="SV2" library="con-lsta" package="FE13-2" value="OPi Zero 2x13" x="25.146" y="2.286" rot="MR180">
 <attribute name="OC_NEWARK" value="unknown" x="25.146" y="2.286" size="1.778" layer="28" rot="MR180" display="off"/>
 <attribute name="MPN" value="" x="25.146" y="2.286" size="1.778" layer="28" rot="MR180" display="off"/>
@@
 <attribute name="OC_FARNELL" value="unknown" x="25.146" y="2.286" size="1.778" layer="28" rot="MR180" display="off"/>
 </element>
-<element name="I2C" library="con-lstb" package="MA04-1" value="" x="5.08" y="11.684" rot="R270">
+<element name="SV3" library="con-lstb" package="MA04-1" value="I2C-OLED" x="5.08" y="11.684" rot="R270">
 <attribute name="OC_NEWARK" value="unknown" x="5.08" y="11.684" size="1.778" layer="27" rot="R270" display="off"/>
 <attribute name="MPN" value="" x="5.08" y="11.684" size="1.778" layer="27" rot="R270" display="off"/>
@@
 <element name="J1" library="adafruit" package="1X2-3.5MM" value="1X2-3.5MM" x="5.08" y="36.068" rot="R270"/>
 <element name="IC1" library="74xx-eu" package="DIL14" value="74HCT125" x="27.94" y="15.748" rot="R90"/>
-<element name="R2" library="rcl" package="0204/7" value="" x="19.05" y="18.288" rot="R90"/>
-<element name="C2" library="rcl" package="E5-6" value="" x="12.7" y="36.83" rot="R90"/>
-<element name="C1" library="rcl" package="E5-6" value="" x="12.7" y="27.432" rot="R270"/>
-<element name="C3" library="rcl" package="C050-024X044" value="" x="29.21" y="26.924"/>
-<element name="JP1" library="pinhead" package="1X02" value="" x="20.32" y="34.29" rot="R180"/>
-<element name="LED1" library="led" package="LED3MM" value="" x="20.32" y="38.862"/>
-<element name="R1" library="rcl" package="0204/7" value="" x="27.94" y="38.862" rot="R180"/>
+<element name="R1" library="rcl" package="0204/7" value="330" x="19.05" y="18.288" rot="R90"/>
+<element name="C2" library="rcl" package="E5-6" value="1000u" x="12.7" y="36.83" rot="R90"/>
+<element name="C1" library="rcl" package="E5-6" value="1000u" x="12.7" y="27.432" rot="R270"/>
+<element name="C3" library="rcl" package="C050-024X044" value="100n" x="29.21" y="26.924"/>
+<element name="JP1" library="pinhead" package="1X02" value="jumper" x="20.32" y="34.29" rot="R180"/>
+<element name="LED1" library="led" package="LED3MM" value="3mm" x="20.32" y="38.862"/>
+<element name="R2" library="rcl" package="0204/7" value="330" x="27.94" y="38.862" rot="R180"/>
 </elements>
 <signals>
 <signal name="GND">
-<contactref element="SV3" pad="6"/>
-<contactref element="I2C" pad="1"/>
-<contactref element="SV3" pad="14"/>
+<contactref element="SV2" pad="6"/>
+<contactref element="SV3" pad="1"/>
+<contactref element="SV2" pad="14"/>
 <contactref element="IC1" pad="13"/>
 <contactref element="IC1" pad="1"/>
 <contactref element="J1" pad="2"/>
 <contactref element="IC1" pad="7"/>
-<contactref element="SV4" pad="2"/>
+<contactref element="SV1" pad="2"/>
 <polygon width="0.4064" layer="16" isolate="0.4064">
 <vertex x="49.022" y="-0.254"/>
@@
 <via x="46.228" y="2.794" extent="1-16" drill="3.2"/>
 <via x="4.064" y="42.926" extent="1-16" drill="3.2"/>
-<contactref element="SV3" pad="25"/>
+<contactref element="SV2" pad="25"/>
 <wire x1="46.228" y1="2.794" x2="45.466" y2="2.794" width="0.4064" layer="16"/>
 <wire x1="45.466" y1="2.794" x2="43.942" y2="1.27" width="0.4064" layer="16"/>
@@
 <vertex x="1.27" y="-0.254"/>
 </polygon>
-<contactref element="SV3" pad="9"/>
-<contactref element="SV3" pad="20"/>
+<contactref element="SV2" pad="9"/>
+<contactref element="SV2" pad="20"/>
 <wire x1="12.7" y1="39.37" x2="5.08" y2="39.37" width="0.4064" layer="16"/>
 <wire x1="12.7" y1="39.37" x2="12.7" y2="40.64" width="0.4064" layer="16"/>
 <wire x1="12.7" y1="40.64" x2="13.97" y2="41.91" width="0.4064" layer="16"/>
-<contactref element="R1" pad="1"/>
+<contactref element="R2" pad="1"/>
 <wire x1="31.75" y1="41.91" x2="13.97" y2="41.91" width="0.4064" layer="16"/>
 <wire x1="31.75" y1="41.91" x2="37.338" y2="41.91" width="0.4064" layer="16"/>
@@
 </signal>
 <signal name="5V">
-<contactref element="SV3" pad="4"/>
-<contactref element="SV3" pad="2"/>
+<contactref element="SV2" pad="4"/>
+<contactref element="SV2" pad="2"/>
 <contactref element="IC1" pad="14"/>
-<contactref element="SV4" pad="1"/>
+<contactref element="SV1" pad="1"/>
 <contactref element="C3" pad="1"/>
 <contactref element="JP1" pad="1"/>
@@
 </signal>
 <signal name="I2C_SDA">
-<contactref element="SV3" pad="3"/>
-<contactref element="I2C" pad="4"/>
+<contactref element="SV2" pad="3"/>
+<contactref element="SV3" pad="4"/>
 <wire x1="12.446" y1="1.016" x2="11.176" y2="2.286" width="0.4064" layer="16"/>
 <wire x1="11.176" y1="2.286" x2="11.176" y2="7.112" width="0.4064" layer="16"/>
@@
 </signal>
 <signal name="I2C_SCL">
-<contactref element="SV3" pad="5"/>
-<contactref element="I2C" pad="3"/>
+<contactref element="SV2" pad="5"/>
+<contactref element="SV3" pad="3"/>
 <wire x1="14.986" y1="1.016" x2="13.716" y2="2.286" width="0.4064" layer="16"/>
 <wire x1="13.716" y1="2.286" x2="13.716" y2="9.144" width="0.4064" layer="16"/>
@@
 </signal>
 <signal name="3V3">
-<contactref element="SV3" pad="1"/>
-<contactref element="I2C" pad="2"/>
+<contactref element="SV2" pad="1"/>
+<contactref element="SV3" pad="2"/>
 <wire x1="9.906" y1="1.016" x2="8.636" y2="1.016" width="0.4064" layer="1"/>
 <wire x1="8.636" y1="1.016" x2="8.128" y2="1.524" width="0.4064" layer="1"/>
@@
 </signal>
 <signal name="SPI_MOSI">
-<contactref element="SV3" pad="19"/>
+<contactref element="SV2" pad="19"/>
 <contactref element="IC1" pad="12"/>
 <wire x1="32.766" y1="1.016" x2="31.496" y2="2.286" width="0.4064" layer="1"/>
@@
 <signal name="MOSI">
 <contactref element="IC1" pad="11"/>
-<contactref element="R2" pad="1"/>
+<contactref element="R1" pad="1"/>
 <wire x1="24.13" y1="15.748" x2="20.32" y2="15.748" width="0.4064" layer="16"/>
 <wire x1="20.32" y1="15.748" x2="19.05" y2="14.478" width="0.4064" layer="16"/>
@@
 <signal name="SPI_CLK">
 <contactref element="IC1" pad="2"/>
-<contactref element="SV3" pad="23"/>
+<contactref element="SV2" pad="23"/>
 <wire x1="37.846" y1="1.016" x2="36.576" y2="2.286" width="0.4064" layer="1"/>
 <wire x1="36.576" y1="2.286" x2="36.576" y2="4.826" width="0.4064" layer="1"/>
@@
 <wire x1="34.036" y1="9.906" x2="33.274" y2="10.668" width="0.4064" layer="1"/>
 <wire x1="33.274" y1="10.668" x2="31.75" y2="10.668" width="0.4064" layer="1"/>
-</signal>
-<signal name="SPI_MISO">
-<contactref element="SV3" pad="21"/>
 </signal>
 <signal name="V+">
@@
 </signal>
 <signal name="N$2">
-<contactref element="R2" pad="2"/>
+<contactref element="R1" pad="2"/>
 <contactref element="CN1" pad="3"/>
 <wire x1="19.05" y1="22.098" x2="18.542" y2="22.606" width="0.4064" layer="1"/>
@@
 <signal name="N$1">
 <contactref element="LED1" pad="K"/>
-<contactref element="R1" pad="2"/>
+<contactref element="R2" pad="2"/>
 <wire x1="21.59" y1="38.862" x2="24.13" y2="38.862" width="0.4064" layer="16"/>
 </signal>
