File: eagle/Orange-Pi-Zero/LTC/P2/zero_board.brd (EAGLE design)
At the start: 47.8 x 46 mm, 17 parts, among them IC1 MCP6002DIP

Commit message: Added new gerber.zip files
Parts:
- removed I2C: (no value), pinhead:1X04
- removed LED'S, SPI: (no value), pinhead:1X05
- added R6: 330, rcl:0204V
- added SV3: OLED, pinhead:1X04
- added SV4: 7SEGMENT, pinhead:1X04
- added SV5: MATRIX, pinhead:1X05
- added SV6: LED, pinhead:1X02
- D1: value (none) -> 3V3
- JP1: value (none) -> L/R
- LED1: value (none) -> 3MM
- SV1: value (none) -> OPI_GPIO
- SV2: value (none) -> OPI_not_used
- SV7: value (none) -> MIDI
- renumbered MIDI to SV7
Connections:
- removed net GPIO18: LED'S.3, SV1.18
- removed net GPIO19: LED'S.4, SV1.16
- removed net GPIO2: LED'S.2, SV1.22
- new net LED_EXT: R6.1, SV6.2
- new net N$4: R6.2, SV1.16
- net 3V3: now also SV3.2, SV4.2; no longer I2C.2, LED'S.5
- net 5V: now also SV5.1; no longer SPI.1
- net GND: now also SV3.1, SV4.1, SV5.2, SV6.1; no longer I2C.1, LED'S.1, SPI.2
- net I2C_SCL: now also SV3.3, SV4.3; no longer I2C.3
- net I2C_SDA: now also SV3.4, SV4.4; no longer I2C.4
- net SPI_CLK: now also SV5.5; no longer SPI.5
- net SPI_CS: now also SV5.4; no longer SPI.4
- net SPI_MOSI: now also SV5.3; no longer SPI.3
Routing:
- net GND: track 137.0 -> 6.64 mm
- net GPIO2: track 15.2 -> 0.00 mm
- net GPIO18: track 14.1 -> 0.00 mm
- net GPIO19: track 14.1 -> 0.00 mm
- net N$4: track 0.00 -> 13.6 mm
- net 3V3: track 58.1 -> 47.0 mm
- net I2C_SDA: track 13.0 -> 21.8 mm
- net SPI_CS: track 39.2 -> 35.3 mm
- net I2C_SCL: track 17.5 -> 21.4 mm, vias 0 -> 1
- net LED_EXT: track 0.00 -> 3.05 mm
- net SPI_MOSI: track 32.9 -> 30.5 mm
- net GPIO10: track 42.1 -> 41.1 mm
- net SPI_CLK: track 41.1 -> 40.2 mm
- net 5V: track 16.4 -> 16.7 mm, vias 0 -> 1
Other:
- board size 47.8 x 46 mm -> 48.8 x 48.3 mm
