File: eagle/Orange-Pi-Zero/Pixel/P5/zero_board.brd (EAGLE design)
At the start: 48.8 x 48.3 mm, 17 parts, among them CN1 1X4-3.5MM, IC1 74HCT125, J1 1X2-3.5MM

Commit message: Pixel 1x 4 Universes SMD board
Parts:
- removed C2: 1000u, rcl:E5-6
- removed C3: 100n, rcl:C050-024X044
- removed J1: 1X2-3.5MM, adafruit:1X2-3.5MM
- removed JP3: LED EXT, pinhead:1X02
- removed LED1: 3mm, led:LED3MM
- removed R3: 330, rcl:R0805
- removed SV2: OPi Zero 2x13, con-lsta:FE13-2
- removed SV3: I2C-OLED, con-lstb:MA04-1
- removed SV4: I2C-7SEGMENT, con-lstb:MA04-1
- C1: value 1000u -> 100n; device rcl:E5-6 -> rcl:C0805
- IC1: value 74HCT125 -> 74LVC2G125DCT; device 74xx-eu:SO14 -> 74xx-little-de:SSOP08
- JP1: value jumper -> (none); device pinhead:1X02 -> pinhead:1X04
- JP2: value Debug -> LED STATUS
- R2: value 330 -> 1K
- SV1: value OPi Zero 1x13 -> OPi Zero 2x13; device con-lsta:FE13 -> con-lsta:FE13-2
- moved SV1 41.9 mm to (25.1, 2.29), turned to 180 degrees
- moved R2 31.9 mm to (25.1, 7.11)
- moved JP1 28.7 mm to (8.64, 8.13), turned to 0 degrees
- moved C1 17.9 mm to (22.1, 12.2)
- moved JP2 13.2 mm to (19.8, 8.13), turned to 180 degrees
- moved CN1 10.1 mm to (8.13, 14.7), turned to 180 degrees
- moved R1 2.84 mm to (18.8, 16.0), turned to 180 degrees
- moved IC1 1.78 mm to (25.9, 12.2), turned to 0 degrees
Connections:
- removed net N$1: LED1.K, R2.2
- removed net N$2: IC1.8, R3.1
- removed net V+: C1.+, C2.+, CN1.1, J1.1, JP1.2, LED1.A
- net 3V3: now also JP1.2, SV1.1; no longer SV2.1, SV3.2, SV4.2
- net 5V: now also C1.1, CN1.1, IC1.8, SV1.2, SV1.4; no longer C3.1, IC1.14, IC1.4, JP1.1, SV1.1, SV2.2, SV2.4
- net CLK: now also CN1.3; no longer CN1.2
- net GND: now also C1.2, IC1.4, JP1.1, SV1.14, SV1.20, SV1.25, SV1.6, SV1.9; no longer C1.-, C2.-, C3.2, IC1.10, IC1.13, J1.2, JP3.2, R2.1, SV1.2, SV2.14, SV2.20, SV2.25, SV2.6, SV2.9, SV3.1, SV4.1
- net I2C_SCL: now also JP1.3, SV1.5; no longer SV2.5, SV3.3, SV4.3
- net I2C_SDA: now also JP1.4, SV1.3; no longer SV2.3, SV3.4, SV4.4
- net MOSI: now also IC1.6; no longer IC1.11
- net N$3: now also JP2.1, R2.2; no longer JP3.1, R3.2
- net OUT: now also CN1.2; no longer CN1.3, JP2.1
- net SPI_CLK: now also IC1.5, SV1.23; no longer IC1.2, SV2.23
- net SPI_MOSI: now also IC1.2, SV1.19; no longer IC1.12, SV2.19
- net STATUS_LED: now also R2.1, SV1.16; no longer IC1.9, SV2.16
Routing:
- net 5V: track 91.1 -> 26.3 mm, vias 1 -> 0
- net V+: track 27.5 -> 0.00 mm
- net CLK: track 46.6 -> 22.5 mm
- net I2C_SDA: track 22.9 -> 8.31 mm
- net OUT: track 22.0 -> 8.91 mm
- net I2C_SCL: track 23.0 -> 10.6 mm, vias 1 -> 0
- net STATUS_LED: track 13.5 -> 4.75 mm, vias 1 -> 0
- net 3V3: track 16.2 -> 8.61 mm
- net N$1: track 5.40 -> 0.00 mm
- net SPI_CLK: track 14.4 -> 18.9 mm
- net N$2: track 3.34 -> 0.00 mm
- net MOSI: track 5.37 -> 8.35 mm
- net SPI_MOSI: track 16.1 -> 14.0 mm
- net N$3: track 4.64 -> 3.77 mm
Other:
- board size 48.8 x 48.3 mm -> 48.8 x 20.1 mm
- board text added: "3V3"
- board text added: "5V"
- board text added: "C"
- board text added: "D"
- board text added: "G"
- board text added: "GND"
- board text added: "SCL"
- board text added: "SDA"
